Commit message: added volatge limit

File: car.urdf (robot description, URDF)
Before this commit: robot rpi_rc_car, 12 links, 11 joints
Links:
- added link base_footprint, mass 0.0001
- added link sonar_rear, mass 0.020; collision box size=0.040 0.020 0.020; visual box size=0.040 0.020 0.020
Joints:
- added joint base_footprint_joint: type fixed, parent base_footprint, child base_link, origin xyz=0 0 0.025 rpy=0 0 0
- added joint sonar_rear_joint: type fixed, parent base_link, child sonar_rear, origin xyz=-0.095 0 0.08 rpy=0 0 3.14159
- joint laser_scanner_joint: limit lower=${-pi/3} upper=${pi/3} effort=1.0 velocity=5.24 -> lower=-1.047197551 upper=1.047197551 effort=1.0 velocity=5.24

Commit message: bug fixes

File: car.urdf (robot description, URDF)
Before this commit: robot rpi_rc_car, 38 links, 37 joints
Links:
- added link servo_arm, mass 0.01; visual box size=0.008 0.040 0.008
- added link tie_rod_left, mass 0.008; visual cylinder length=0.070 radius=0.003
- added link tie_rod_right, mass 0.008; visual cylinder length=0.070 radius=0.003
- link steering_servo: geometry visual box size=0.040 0.020 0.036; visual cylinder length=0.010 radius=0.006
Joints:
- added joint servo_arm_joint: type revolute, parent steering_servo, child servo_arm, origin xyz=0 0 0.028 rpy=0 0 0, axis 0 0 1, limit lower=-0.5236 upper=0.5236 effort=2.0 velocity=3.0
- added joint tie_rod_left_joint: type fixed, parent servo_arm, child tie_rod_left, origin xyz=0 0.020 0 rpy=0 0 0
- added joint tie_rod_right_joint: type fixed, parent servo_arm, child tie_rod_right, origin xyz=0 -0.020 0 rpy=0 0 0
- joint camera_gimbal_base_joint: origin xyz=0.072 -0.022 0.048 rpy=0 0 0 -> xyz=0.105 0.000 0.050 rpy=0 0 0
- joint laser_scanner_joint: origin xyz=0.024 -0.017 0.008 rpy=0 0 0 -> xyz=0.010 0 0.032 rpy=0 0 0; parent camera_tilt_link -> steering_servo
- joint steering_servo_joint: origin xyz=0.080 0 -0.018 rpy=0 0 0 -> xyz=0.105 0 0.0015 rpy=0 0 0
